File: kicad.kicad_sch (KiCad schematic)
At the start: 14 parts, among them U1 1533ir35, U10 74LS245, U11 74LS245, U2 155ll1, U3 155ln1, U4 155tm2, U5 155kp12, U6 155kp11, U7 155kp11, U8 155kp11, U9 155ll1

Commit message: not finish
Parts:
- removed unit 6 of U3
- removed unit 5 of U3
- removed unit 3 of U3
- removed unit 4 of U3
- removed unit 2 of U4
- added C10, C11, C12, C13, C14, C15, C4, C5, C6, C7, C8, C9: 0.1uF, Capacitor_THT:C_Axial_L3.8mm_D2.6mm_P7.50mm_Horizontal, symbol Device:C
- added J2: Keyboard, symbol Connector:Conn_01x20_Pin
- added RN1: R_Network04, Resistor_THT:R_Array_SIP5, symbol Device:R_Network04
- added U12, U13: 537РУ10, Package_DIP:DIP-24_18.0mmx34.29mm_W15.24mm, symbol Memory_RAM:M48Tx2
- added U14: HM628128, Package_DIP:DIP-32_W15.24mm_LongPads, symbol Memory_RAM:HM628128D_DIP32_SOP32
- added U15, U19: 573РФ5, symbol User:2716
- added U17: 155ИР37, symbol 74xx:74LS574
- added U22: 155КП11, symbol 74xx:74LS257
- C1: value 1uF ? -> 1uF
- U1: value 1533ir35 -> 1533ИР35; Analogs (none) -> 74ALS273
- U10, U11: value 74LS245 -> 155АП6; Analogs (none) -> 74245
- U2, U9: value 155ll1 -> 155ЛЛ1; Analogs (none) -> 7432
- U3: value 155ln1 -> 155ЛН1; Analogs (none) -> 7404
- U4: value 155tm2 -> 155ТМ2; Analogs (none) -> 7474
- U5: value 155kp12 -> 155КП12; Analogs (none) -> 74253
- U6, U7, U8: value 155kp11 -> 155КП11; Analogs (none) -> 74257
Connections:
- net +5V: now also C10.1, C11.1, C12.1, C13.1, C14.1, C15.1, C4.1, C5.1, C6.1, C7.1, C8.1, C9.1, J2.3 (Pin_3), J2.4 (Pin_4), U12.24 (VCC), U13.24 (VCC), U14.30 (CS2/CE2), U14.32 (VCC), U15.21 (VPP), U15.24 (VCC), U17.20 (VCC), U19.21 (VPP), U19.24 (VCC), U22.16 (VCC)
- net A0: now also J2.8 (Pin_8), U14.12 (A0), U15.8 (A0)
- net A1: now also J2.7 (Pin_7), U14.11 (A1), U15.7 (A1)
- net A10: now also U14.23 (A10), U15.19 (A10)
- net A11: now also U3.3, U14.25 (A11)
- net A2: now also J2.6 (Pin_6), U14.10 (A2), U15.6 (A2)
- net A3: now also J2.5 (Pin_5), U14.9 (A3), U15.5 (A3)
- net A4: now also U14.8 (A4), U15.4 (A4)
- net A5: now also U14.7 (A5), U15.3 (A5)
- net A6: now also U14.6 (A6), U15.2 (A6)
- net A7: now also U14.5 (A7), U15.1 (A7)
- net A8: now also U14.27 (A8), U15.23 (A8)
- net A9: now also U14.26 (A9), U15.22 (A9)
- net D0: now also J2.13 (Pin_13), U14.13 (I/O0), U15.9 (DQ0)
- net D1: now also J2.14 (Pin_14), U14.14 (I/O1), U15.10 (DQ1)
- net D2: now also J2.15 (Pin_15), U14.15 (I/O2), U15.11 (DQ2)
- net D3: now also J2.16 (Pin_16), U14.17 (I/O3), U15.13 (DQ3)
- net D4: now also J2.17 (Pin_17), U14.18 (I/O4), U15.14 (DQ4)
- net D5: now also J2.18 (Pin_18), U14.19 (I/O5), U15.15 (DQ5)
- net D6: now also J2.19 (Pin_19), U14.20 (I/O6), U15.16 (DQ6)
- net D7: now also J2.20 (Pin_20), U14.21 (I/O7), U15.17 (DQ7)
- net GND: now also C10.2, C11.2, C12.2, C13.2, C14.2, C15.2, C4.2, C5.2, C6.2, C7.2, C8.2, C9.2, J2.1 (Pin_1), J2.2 (Pin_2), RN1.1 (common), U12.12 (VSS), U12.18 (~{E}), U12.20 (~{G}), U13.12 (VSS), U13.18 (~{E}), U13.20 (~{G}), U14.16 (GND), U14.2 (A16), U15.12 (GND), U17.10 (GND), U19.12 (GND), U22.8 (GND)
- net MA0: now also U12.8 (A0), U13.8 (A0)
- net MA1: now also U12.7 (A1), U13.7 (A1)
- net MA10: now also U12.19 (A10), U13.19 (A10)
- net MA2: now also U12.6 (A2), U13.6 (A2)
- net MA3: now also U12.5 (A3), U13.5 (A3)
- net MA4: now also U12.4 (A4), U13.4 (A4)
- net MA5: now also U12.3 (A5), U13.3 (A5)
- net MA6: now also U12.2 (A6), U13.2 (A6)
- net MA7: now also U12.1 (A7), U13.1 (A7)
- net MA8: now also U12.23 (A8), U13.23 (A8)
- net MA9: now also U12.22 (A9), U13.22 (A9)
- net MD0: now also U12.9 (DQ0), U19.5 (A3)
- net MD1: now also U12.10 (DQ1), U19.4 (A4)
- net MD2: now also U12.11 (DQ2), U19.3 (A5)
- net MD3: now also U12.13 (DQ3), U19.2 (A6)
- net MD4: now also U12.14 (DQ4), U19.1 (A7)
- net MD5: now also U12.15 (DQ5), U19.23 (A8)
- net MD6: now also U12.16 (DQ6), U19.22 (A9)
- net MD7: now also U12.17 (DQ7), U19.19 (A10)
- net ROM0: now also U2.9
- net ROMF: now also U2.4
- net /CW: now also U13.21 (~{W})
- net /JW: now also J2.12 (Pin_12)
- net /MR: now also U2.10, U2.5, U14.24 (~{OE})
- net /MW: now also U14.29 (~{WE})
- net /SW: now also U12.21 (~{W})
- net at U3.4: now also U2.2
- net MONITOR0_CS: now reaches U2.8
- net /F000h: now reaches U2.1
- net /F800h: now reaches U2.3
- net /F800h: now also U15.20 (~{OE})
- net at U2.6: now also U15.18 (~{CE})
- new net A12: U14.31 (A15)
- new net A13: U14.28 (A13)
- new net A14: U14.4 (A12)
- new net A15: U14.3 (A14)
- new net G0: U19.8 (A0)
- new net G1: U19.7 (A1)
- new net G2: U19.6 (A2)
- new net INV: U22.1 (S)
- new net LOAD: U17.11 (Cp)
- new net MC0: U13.9 (DQ0), U17.2 (D0)
- new net MC1: U13.10 (DQ1), U17.3 (D1)
- new net MC2: U13.11 (DQ2), U17.4 (D2)
- new net MC3: U13.13 (DQ3), U17.5 (D3)
- new net MC4: U13.14 (DQ4), U17.6 (D4)
- new net MC5: U13.15 (DQ5), U17.7 (D5)
- new net MC6: U13.16 (DQ6), U17.8 (D6)
- new net MC7: U13.17 (DQ7), U17.9 (D7)
- new net RES: J2.11 (Pin_11)
- new net VB: U22.4 (Za)
- new net VD0: U19.9 (DQ0)
- new net VD1: U19.10 (DQ1)
- new net VD2: U19.11 (DQ2)
- new net VD3: U19.13 (DQ3)
- new net VD4: U19.14 (DQ4)
- new net VD5: U19.15 (DQ5)
- new net VG: U22.12 (Zc)
- new net VQA0: U17.19 (Q0), U22.2 (I0a)
- new net VQA1: U17.18 (Q1), U22.3 (I1a)
- new net VQA2: U17.17 (Q2), U22.5 (I0b)
- new net VQA3: U17.16 (Q3), U22.6 (I1b)
- new net VQB0: RN1.5 (R4), U17.15 (Q4), U22.14 (I0c)
- new net VQB1: RN1.4 (R3), U17.14 (Q5), U22.13 (I1c)
- new net VQB2: RN1.3 (R2), U17.13 (Q6), U22.11 (I0d)
- new net VQB3: RN1.2 (R1), U17.12 (Q7), U22.10 (I1d)
- new net VR: U22.7 (Zb)
- new net VY: U22.9 (Zd)
- new net /0000h: J2.9 (Pin_9)
- new net /COLOREN: U17.1 (OE)
- new net /GEN: U19.18 (~{CE}), U19.20 (~{OE}), U22.15 (OE)
- new net /JR: J2.10 (Pin_10)
- new net /RAMCS: U14.22 (~{CS1}/~{CE1})
- no-connect marks 12 -> 14
Other:
- added sheet page2 (page2.kicad_sch)
- company: (none) -> Eugene Chertikhin
- title: (none) -> UT88 display board
- moved on the sheet: U2A, U2B, U2C, U3B

Commit message: finish with 1 question
Parts:
- removed R1: R?, Resistor_THT:R_Axial_DIN0204_L3.6mm_D1.6mm_P5.08mm_Horizontal, symbol Device:R
- removed U1: 1533ИР35, symbol User:74ALS273
- added C16, C17, C18: 0.1uF, Capacitor_THT:C_Axial_L3.8mm_D2.6mm_P7.50mm_Horizontal, symbol Device:C
- added R4: 1k, Resistor_THT:R_Axial_DIN0204_L3.6mm_D1.6mm_P5.08mm_Horizontal, symbol Device:R
- added R40: 10k, Resistor_THT:R_Axial_DIN0204_L3.6mm_D1.6mm_P5.08mm_Horizontal, symbol Device:R
- added U1: 1533ИР35, Package_DIP:DIP-20_W7.62mm_LongPads, symbol 74xx:74LS273
- C1: value 1uF -> 1uF 16V
- R3: value R? -> 10k
- RN1: value R_Network04 -> 10k
Connections:
- net +5V: now also C16.1, C17.1, C18.1, R4.2, R40.2, U1.20 (VCC); no longer U14.30 (CS2/CE2)
- net D0: now also U1.3 (D0)
- net D1: now also U1.4 (D1)
- net D2: now also U1.7 (D2)
- net D3: now also U1.8 (D3)
- net GENSYM: now also U1.2 (Q0)
- net GND: now also C16.2, C17.2, C18.2, U1.10 (GND)
- net ROM0: now also U1.6 (Q2)
- net ROMF: now also U1.9 (Q3)
- net at C1.1, R3.1: now also U1.1 (~{Mr})
- net at U2.11: now also U1.11 (Cp)
- net at U5.14 (A0): now also U1.5 (Q1)
- net at U4.1 (~{R}), U4.4 (~{S}): now also R4.1
- new net: R40.1, U14.30 (CS2/CE2)
Other:
- moved on the sheet: C1, C11, C12, C13, C14, C15

Commit message: update footprint
Parts:
- RN1: value 10k -> 5k
- U10, U11, U17: footprint (none) -> Package_DIP:DIP-20_W7.62mm_LongPads
- U15, U19: footprint (none) -> Package_DIP:DIP-24_18.0mmx34.29mm_W15.24mm_LongPads
- U2, U3, U4, U9: footprint (none) -> Package_DIP:DIP-14_W7.62mm_LongPads
- U22, U5, U6, U7, U8: footprint (none) -> Package_DIP:DIP-16_W7.62mm_LongPads
Changed lines of the file:
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@@
 			)
 		)
-		(property "Footprint" ""
+		(property "Footprint" "Package_DIP:DIP-24_18.0mmx34.29mm_W15.24mm_LongPads"
 			(at 260.35 46.99 0)
 			(effects
@@
 					(size 1.524 1.524)
 				)
+				(hide yes)
 			)
 		)
@@
 			)
 		)
-		(property "Footprint" ""
+		(property "Footprint" "Package_DIP:DIP-14_W7.62mm_LongPads"
 			(at 135.89 133.35 0)
 			(effects
@@
 			)
 		)
-		(property "Footprint" ""
+		(property "Footprint" "Package_DIP:DIP-14_W7.62mm_LongPads"
 			(at 127 170.18 0)
 			(effects
@@
 			)
 		)
-		(property "Footprint" ""
+		(property "Footprint" "Package_DIP:DIP-14_W7.62mm_LongPads"
 			(at 30.48 153.67 0)
 			(effects
@@
 			)
 		)
-		(property "Footprint" ""
+		(property "Footprint" "Package_DIP:DIP-14_W7.62mm_LongPads"
 			(at 120.65 130.81 0)
 			(effects
@@
 			)
 		)
-		(property "Footprint" ""
+		(property "Footprint" "Package_DIP:DIP-24_18.0mmx34.29mm_W15.24mm_LongPads"
 			(at 209.55 46.99 0)
 			(effects
@@
 					(size 1.524 1.524)
 				)
+				(hide yes)
 			)
 		)
@@
 			)
 		)
-		(property "Footprint" ""
+		(property "Footprint" "Package_DIP:DIP-20_W7.62mm_LongPads"
 			(at 201.93 91.44 0)
 			(effects
@@
 			)
 		)
-		(property "Footprint" ""
+		(property "Footprint" "Package_DIP:DIP-20_W7.62mm_LongPads"
 			(at 74.93 96.52 0)
 			(effects
@@
 			)
 		)
-		(property "Footprint" ""
+		(property "Footprint" "Package_DIP:DIP-14_W7.62mm_LongPads"
 			(at 125.73 187.96 0)
 			(effects
@@
 			)
 		)
-		(property "Footprint" ""
+		(property "Footprint" "Package_DIP:DIP-14_W7.62mm_LongPads"
 			(at 135.89 142.24 0)
 			(effects
@@
 			)
 		)
-		(property "Footprint" ""
+		(property "Footprint" "Package_DIP:DIP-14_W7.62mm_LongPads"
 			(at 63.5 187.96 0)
 			(effects
@@
 			)
 		)
-		(property "Footprint" ""
+		(property "Footprint" "Package_DIP:DIP-14_W7.62mm_LongPads"
 			(at 158.75 187.96 0)
 			(effects
@@
 			)
 		)
-		(property "Footprint" ""
+		(property "Footprint" "Package_DIP:DIP-14_W7.62mm_LongPads"
 			(at 127 157.48 0)
 			(effects
@@
 			)
 		)
-		(property "Footprint" ""
+		(property "Footprint" "Package_DIP:DIP-14_W7.62mm_LongPads"
 			(at 142.24 167.64 0)
 			(effects
@@
 			)
 		)
-		(property "Footprint" ""
+		(property "Footprint" "Package_DIP:DIP-16_W7.62mm_LongPads"
 			(at 97.79 148.59 0)
 			(effects
@@
 			)
 		)
-		(property "Footprint" ""
+		(property "Footprint" "Package_DIP:DIP-14_W7.62mm_LongPads"
 			(at 154.94 135.89 0)
 			(effects
@@
 			)
 		)
-		(property "Value" "10k"
+		(property "Value" "5k"
 			(at 269.494 73.66 90)
 			(effects
@@
 			)
 		)
-		(property "Footprint" ""
+		(property "Footprint" "Package_DIP:DIP-16_W7.62mm_LongPads"
 			(at 245.11 93.98 0)
 			(effects
@@
 			)
 		)
-		(property "Footprint" ""
+		(property "Footprint" "Package_DIP:DIP-14_W7.62mm_LongPads"
 			(at 154.94 144.78 0)
 			(effects
@@
 			)
 		)
-		(property "Footprint" ""
+		(property "Footprint" "Package_DIP:DIP-14_W7.62mm_LongPads"
 			(at 95.25 187.96 0)
 			(effects
@@
 			)
 		)
-		(property "Footprint" ""
+		(property "Footprint" "Package_DIP:DIP-16_W7.62mm_LongPads"
 			(at 35.56 39.37 0)
 			(effects
@@
 			)
 		)
-		(property "Footprint" ""
+		(property "Footprint" "Package_DIP:DIP-16_W7.62mm_LongPads"
 			(at 116.84 39.37 0)
 			(effects
@@
 			)
 		)
-		(property "Footprint" ""
+		(property "Footprint" "Package_DIP:DIP-20_W7.62mm_LongPads"
 			(at 34.29 96.52 0)
 			(effects
@@
 			)
 		)
-		(property "Footprint" ""
+		(property "Footprint" "Package_DIP:DIP-14_W7.62mm_LongPads"
 			(at 30.48 185.42 0)
 			(effects
@@
 			)
 		)
-		(property "Footprint" ""
+		(property "Footprint" "Package_DIP:DIP-14_W7.62mm_LongPads"
 			(at 182.88 68.58 0)
 			(effects
@@
 			)
 		)
-		(property "Footprint" ""
+		(property "Footprint" "Package_DIP:DIP-16_W7.62mm_LongPads"
 			(at 73.66 39.37 0)
 			(effects
