File: page2.kicad_sch (KiCad schematic)
At the start: 46 parts, among them J1 Conn_01x02_Pin, Q1 КТ315, Q2 КТ315, Q3 КТ315, Q4 КТ315, U16 155ИЕ4, U18 155ЛА3, U20 155ИЕ5, U21 155ЛА1, U23 155ИР13, U24 155КП12, U25 155ЛЛ1, U26 155ЛН1, U27 155ЛП5, U28 155ИЕ5, U29 155ЛА1, U3 155ЛН1, U30 155ИМ3, U31 155ЛП5, U32 155ИЕ2, U33 155ИЕ5, U4 155ТМ2

Commit message: finish with 1 question
Parts:
- removed C3: 10uF 16v ?, Capacitor_THT:C_Axial_L3.8mm_D2.6mm_P7.50mm_Horizontal, symbol Device:C
- removed J1: Conn_01x02_Pin, Connector_Wire:SolderWire-1.5sqmm_1x02_P7.8mm_D1.7mm_OD3.9mm, symbol Connector:Conn_01x02_Pin
- removed Q1, Q2, Q3, Q4: КТ315, Package_TO_SOT_THT:TO-3P-3_Vertical, symbol Transistor_BJT:2N3055
- added C3: 10uF 16V, Capacitor_THT:CP_Axial_L10.0mm_D4.5mm_P15.00mm_Horizontal, symbol Device:C_Polarized
- added Q1, Q2, Q3, Q4, Q5: КТ315A, Package_TO_SOT_THT:TO-39-3, symbol Transistor_BJT:2N3904
- added R16, R17, R18, R19, R26, R30: 1k, Resistor_THT:R_Axial_DIN0204_L3.6mm_D1.6mm_P5.08mm_Horizontal, symbol Device:R
- added R23: 680, Resistor_THT:R_Axial_DIN0204_L3.6mm_D1.6mm_P5.08mm_Horizontal, symbol Device:R
- added R24: 2k, Resistor_THT:R_Axial_DIN0204_L3.6mm_D1.6mm_P5.08mm_Horizontal, symbol Device:R
- added R25, R27, R29, R31: 200, Resistor_THT:R_Axial_DIN0204_L3.6mm_D1.6mm_P5.08mm_Horizontal, symbol Device:R
- added R28: 470, Resistor_THT:R_Axial_DIN0204_L3.6mm_D1.6mm_P5.08mm_Horizontal, symbol Device:R
- added R32: 27, Resistor_THT:R_Axial_DIN0204_L3.6mm_D1.6mm_P5.08mm_Horizontal, symbol Device:R
- added SW1: Priority Cpu/Video, symbol Switch:SW_DIP_x01
- added SW2: Video settings, symbol Switch:SW_DIP_x04
- D1: renamed from D3; value D -> 1n4148
- D2: value D -> 1n4148
- D3: renamed from D1; value D -> 1n4148
- R2: value 10k -> 1k
- R39: value R -> 1k
- renumbered R4 to R15, R22 to R20, R5 to R21, R6 to R22, R15 to R33, R8 to R34, R7 to R35, R38 to R36, R36 to R38
Connections:
- net +5V: now also Q1.3 (C), Q2.3 (C), Q3.3 (C), Q4.3 (C), Q5.3 (C), R16.1, R17.1, R18.2, R19.2, R23.2
- net G3: now also U26.1
- net GND: now also R25.1, R27.1, R29.1, R30.1, R31.1, SW2.1, SW2.2, SW2.3, SW2.4
- net RD: now also SW1.1
- net VIDEO1: now also C3.1
- net at R22.2, R38.2: now also Q2.2 (B)
- net at R33.1: now also Q2.1 (E), R28.1, R29.2
- net at C2.2, R14.1, R15.2: now also C3.2
- net at U31.5: now also R18.1, SW2.5
- net at R21.2, R37.2: now also Q3.2 (B)
- net DIVCP0: now reaches U16.8 (Q3), U18.4, U20.14 (CP0)
- net at U31.2: now also R19.1, SW2.8
- net at R14.2: now also Q1.1 (E)
- net at U31.10: now also R17.2, SW2.6
- net at R20.2, R36.2: now also Q4.2 (B)
- net at R35.1: now also Q4.1 (E), R24.1, R25.2
- net at R11.2, R12.2, R13.1: now also Q1.2 (B)
- net at R34.1: now also Q3.1 (E), R26.1, R27.2
- net at U30.15 (S4): now also U26.3; no longer U26.1
- net at U31.12: now also R16.2, SW2.7
- net at U25.3: now also SW1.2
- net CP1Q0: now reaches U20.1 (CP1..3), U20.12 (Q0)
- new net: Q5.2 (B), R23.1, R24.2, R26.2, R28.2, R30.2
- new net: Q5.1 (E), R31.2, R32.2
- new net VIDEO2: R32.1
- no-connect marks 16 -> 30
Other:
- moved on the sheet: C2, D1, D2, D3, R1, R10, R11, R12, R13, R14, R15, R20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

Commit message: update footprint
Parts:
- U16, U18, U20, U21, U25, U26, U27, U28, U29, U3, U31, U32, U33, U4: footprint (none) -> Package_DIP:DIP-14_W7.62mm_LongPads
- U23: footprint (none) -> Package_DIP:DIP-24_18.0mmx34.29mm_W15.24mm_LongPads
- U24, U30: footprint (none) -> Package_DIP:DIP-16_W7.62mm_LongPads
Changed lines of the file:
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@@
 			)
 		)
-		(property "Footprint" ""
+		(property "Footprint" "Package_DIP:DIP-14_W7.62mm_LongPads"
 			(at 76.2 36.83 0)
 			(effects
@@
 			)
 		)
-		(property "Footprint" ""
+		(property "Footprint" "Package_DIP:DIP-14_W7.62mm_LongPads"
 			(at 93.98 39.37 0)
 			(effects
@@
 			)
 		)
-		(property "Footprint" ""
+		(property "Footprint" "Package_DIP:DIP-14_W7.62mm_LongPads"
 			(at 156.21 83.82 0)
 			(effects
@@
 			)
 		)
-		(property "Footprint" ""
+		(property "Footprint" "Package_DIP:DIP-14_W7.62mm_LongPads"
 			(at 161.29 115.57 0)
 			(effects
@@
 			)
 		)
-		(property "Footprint" ""
+		(property "Footprint" "Package_DIP:DIP-14_W7.62mm_LongPads"
 			(at 195.58 40.64 0)
 			(effects
@@
 			)
 		)
-		(property "Footprint" ""
+		(property "Footprint" "Package_DIP:DIP-14_W7.62mm_LongPads"
 			(at 59.69 168.91 0)
 			(effects
@@
 			)
 		)
-		(property "Footprint" ""
+		(property "Footprint" "Package_DIP:DIP-14_W7.62mm_LongPads"
 			(at 33.02 91.44 0)
 			(effects
@@
 			)
 		)
-		(property "Footprint" ""
+		(property "Footprint" "Package_DIP:DIP-14_W7.62mm_LongPads"
 			(at 26.67 191.77 0)
 			(effects
@@
 			)
 		)
-		(property "Footprint" ""
+		(property "Footprint" "Package_DIP:DIP-14_W7.62mm_LongPads"
 			(at 110.49 86.36 0)
 			(effects
@@
 			)
 		)
-		(property "Footprint" ""
+		(property "Footprint" "Package_DIP:DIP-14_W7.62mm_LongPads"
 			(at 203.2 123.19 0)
 			(effects
@@
 			)
 		)
-		(property "Footprint" ""
+		(property "Footprint" "Package_DIP:DIP-14_W7.62mm_LongPads"
 			(at 106.68 179.07 0)
 			(effects
@@
 			)
 		)
-		(property "Footprint" ""
+		(property "Footprint" "Package_DIP:DIP-14_W7.62mm_LongPads"
 			(at 137.16 110.49 0)
 			(effects
@@
 			)
 		)
-		(property "Footprint" ""
+		(property "Footprint" "Package_DIP:DIP-14_W7.62mm_LongPads"
 			(at 195.58 30.48 0)
 			(effects
@@
 			)
 		)
-		(property "Footprint" ""
+		(property "Footprint" "Package_DIP:DIP-14_W7.62mm_LongPads"
 			(at 57.15 67.31 0)
 			(effects
@@
 			)
 		)
-		(property "Footprint" ""
+		(property "Footprint" "Package_DIP:DIP-14_W7.62mm_LongPads"
 			(at 106.68 191.77 0)
 			(effects
@@
 			)
 		)
-		(property "Footprint" ""
+		(property "Footprint" "Package_DIP:DIP-14_W7.62mm_LongPads"
 			(at 142.24 179.07 0)
 			(effects
@@
 			)
 		)
-		(property "Footprint" ""
+		(property "Footprint" "Package_DIP:DIP-14_W7.62mm_LongPads"
 			(at 124.46 179.07 0)
 			(effects
@@
 			)
 		)
-		(property "Footprint" ""
+		(property "Footprint" "Package_DIP:DIP-14_W7.62mm_LongPads"
 			(at 29.21 180.34 0)
 			(effects
@@
 			)
 		)
-		(property "Footprint" ""
+		(property "Footprint" "Package_DIP:DIP-14_W7.62mm_LongPads"
 			(at 44.45 180.34 0)
 			(effects
@@
 			)
 		)
-		(property "Footprint" ""
+		(property "Footprint" "Package_DIP:DIP-14_W7.62mm_LongPads"
 			(at 53.34 191.77 0)
 			(effects
@@
 			)
 		)
-		(property "Footprint" ""
+		(property "Footprint" "Package_DIP:DIP-14_W7.62mm_LongPads"
 			(at 133.35 191.77 0)
 			(effects
@@
 			)
 		)
-		(property "Footprint" ""
+		(property "Footprint" "Package_DIP:DIP-14_W7.62mm_LongPads"
 			(at 226.06 130.81 0)
 			(effects
@@
 			)
 		)
-		(property "Footprint" ""
+		(property "Footprint" "Package_DIP:DIP-14_W7.62mm_LongPads"
 			(at 229.87 85.09 0)
 			(effects
@@
 			)
 		)
-		(property "Footprint" ""
+		(property "Footprint" "Package_DIP:DIP-14_W7.62mm_LongPads"
 			(at 265.43 128.27 0)
 			(effects
@@
 			)
 		)
-		(property "Footprint" ""
+		(property "Footprint" "Package_DIP:DIP-14_W7.62mm_LongPads"
 			(at 195.58 52.07 0)
 			(effects
@@
 			)
 		)
-		(property "Footprint" ""
+		(property "Footprint" "Package_DIP:DIP-14_W7.62mm_LongPads"
 			(at 160.02 191.77 0)
 			(effects
@@
 			)
 		)
-		(property "Footprint" ""
+		(property "Footprint" "Package_DIP:DIP-16_W7.62mm_LongPads"
 			(at 58.42 100.33 0)
 			(effects
@@
 			)
 		)
-		(property "Footprint" ""
+		(property "Footprint" "Package_DIP:DIP-14_W7.62mm_LongPads"
 			(at 139.7 83.82 0)
 			(effects
@@
 			)
 		)
-		(property "Footprint" ""
+		(property "Footprint" "Package_DIP:DIP-14_W7.62mm_LongPads"
 			(at 36.83 85.09 0)
 			(effects
@@
 			)
 		)
-		(property "Footprint" ""
+		(property "Footprint" "Package_DIP:DIP-14_W7.62mm_LongPads"
 			(at 218.44 99.06 0)
 			(effects
@@
 			)
 		)
-		(property "Footprint" ""
+		(property "Footprint" "Package_DIP:DIP-14_W7.62mm_LongPads"
 			(at 33.02 76.2 0)
 			(effects
@@
 			)
 		)
-		(property "Footprint" ""
+		(property "Footprint" "Package_DIP:DIP-14_W7.62mm_LongPads"
 			(at 195.58 62.23 0)
 			(effects
@@
 			)
 		)
-		(property "Footprint" ""
+		(property "Footprint" "Package_DIP:DIP-14_W7.62mm_LongPads"
 			(at 44.45 171.45 0)
 			(effects
@@
 			)
 		)
-		(property "Footprint" ""
+		(property "Footprint" "Package_DIP:DIP-14_W7.62mm_LongPads"
 			(at 67.31 57.15 0)
 			(effects
@@
 			)
 		)
-		(property "Footprint" ""
+		(property "Footprint" "Package_DIP:DIP-14_W7.62mm_LongPads"
 			(at 80.01 191.77 0)
 			(effects
@@
 			)
 		)
-		(property "Footprint" ""
+		(property "Footprint" "Package_DIP:DIP-14_W7.62mm_LongPads"
 			(at 245.11 96.52 0)
 			(effects
@@
 			)
 		)
-		(property "Footprint" ""
+		(property "Footprint" "Package_DIP:DIP-14_W7.62mm_LongPads"
 			(at 229.87 93.98 0)
 			(effects
@@
 			)
 		)
-		(property "Footprint" ""
+		(property "Footprint" "Package_DIP:DIP-14_W7.62mm_LongPads"
 			(at 48.26 160.02 0)
 			(effects
@@
 			)
 		)
-		(property "Footprint" ""
+		(property "Footprint" "Package_DIP:DIP-14_W7.62mm_LongPads"
 			(at 80.01 179.07 0)
 			(effects
@@
 			)
 		)
-		(property "Footprint" ""
+		(property "Footprint" "Package_DIP:DIP-14_W7.62mm_LongPads"
 			(at 93.98 29.21 0)
 			(effects
@@
 			)
 		)
-		(property "Footprint" ""
+		(property "Footprint" "Package_DIP:DIP-14_W7.62mm_LongPads"
 			(at 69.85 26.67 0)
 			(effects
@@
 			)
 		)
-		(property "Footprint" ""
+		(property "Footprint" "Package_DIP:DIP-14_W7.62mm_LongPads"
 			(at 100.33 115.57 0)
 			(effects
@@
 			)
 		)
-		(property "Footprint" ""
+		(property "Footprint" "Package_DIP:DIP-14_W7.62mm_LongPads"
 			(at 160.02 179.07 0)
 			(effects
@@
 			)
 		)
-		(property "Footprint" ""
+		(property "Footprint" "Package_DIP:DIP-14_W7.62mm_LongPads"
 			(at 187.96 120.65 0)
 			(effects
@@
 			)
 		)
-		(property "Footprint" ""
+		(property "Footprint" "Package_DIP:DIP-16_W7.62mm_LongPads"
 			(at 196.85 93.98 0)
 			(effects
@@
 			)
 		)
-		(property "Footprint" ""
+		(property "Footprint" "Package_DIP:DIP-24_18.0mmx34.29mm_W15.24mm_LongPads"
 			(at 38.1 39.37 0)
 			(effects
@@
 					(size 1.524 1.524)
 				)
+				(hide yes)
 			)
 		)
